File: picareta_schem/picareta_schem.kicad_sch (KiCad schematic)
At the start: 17 parts, among them M1 Motor, M2 Motor, M3 Motor

Commit message: Relatorio update
Parts:
- renumbered SENTERA_6X_CAMERA to MICASENSE_REDEDGE-P
Connections:
- net PAYLOAD_SELECT: now also JetsonOrinNX8GB2.95 (SPI0_CS0); no longer JetsonOrinNX8GB2.97 (SPI0_CS1)
- net SPI_CLK: no longer MatekH743-WLITE1. (3V3)
- net SPI_MISO: no longer MatekH743-WLITE1. (3V3)
- net SPI_MOSI: no longer MatekH743-WLITE1. (3V3)
- new net: M3., U5. (W) (x2)
- new net: JetsonOrinNX8GB2.118 (GPIO01_), MICASENSE_REDEDGE-P. (VDD-)
- new net: JetsonOrinNX8GB2.207 (GPIO07_PWM), MICASENSE_REDEDGE-P. (VDD-)
- new net: M1., U1. (BAT-) (x2)
- new net: ADS1220. (AIN3), FLC3-1. (Z_A3) (x3)
- new net: U1. (BAT-), U3. (BAT-), U4. (Cur), U5. (W) (x2)
- new net: M2., U3. (BAT-) (x2)
- new net: JetsonOrinNX8GB2.101 (UART0_RXD), MatekH743-WLITE1.PA10 (RX1)
- new net: JetsonOrinNX8GB2.218 (GPIO12), MatekH743-WLITE1.PB0 (S1)
- new net: JetsonOrinNX8GB2.99 (UART0_TXD_), MatekH743-WLITE1.PA9 (TX1)
- new net: M10Q5883. (GND), MatekH743-WLITE1.PB6 (CL1)
- new net: M10Q5883. (GND), MatekH743-WLITE1.PB7 (DA1)
- new net: M10Q5883. (GND), MatekH743-WLITE1.PD5 (TX2)
- new net: M10Q5883. (GND), MatekH743-WLITE1.PD6 (RX2)
- no-connect marks 21 -> 20
Other:
- note added: "Omniscan Electronics Schematic"
- moved on the sheet: MatekH743-WLITE1
